Commit message: Add AGX sensor calibration test and enhance joint control
- Introduced a new script for AGX sensor calibration testing, validating RGB-D camera configurations and outputs.
- Implemented a method in the SteeringDriveController to release hold on specified joints, allowing external control during acceptance tests.

File: src/ros2_car_model_ws/src/1557/urdf/1557_all.urdf (robot description, URDF)
Before this commit: robot ranger_with_xarm6, 31 links, 30 joints
Joints:
- joint lifting_joint: origin xyz=0 0 0 rpy=0 0 0 -> xyz=0 0 0.15 rpy=0 0 0
- joint pan_tilt_joint: origin xyz=-0.12 -0.002 0.8 rpy=0 0 0 -> xyz=-0.12 -0.002 0.95 rpy=0 0 0
- joint ranger_with_xarm: origin xyz=-0.08 -0.01 0.646  rpy=0 -1.57 3.14 -> xyz=-0.08 -0.01 0.796  rpy=0 -1.57 3.14
